File: pcb/te96.kicad_pcb (KiCad board)
At the start: 2 copper layers, 100 x 100 mm, 254 parts, among them J1 Conn_02x08_Top_Bottom, J10 Conn_01x04, J2 Conn_02x08_Top_Bottom, J3 MJ-4PP-9, J4 MJ-4PP-9, J7 Conn_01x03, J8 Conn_01x03, J9 Conn_01x04, SW1 SW_and_D, SW10 SW_and_D, SW11 SW_and_D, SW12 SW_and_D, SW13 SW_and_D, SW14 SW_and_D, SW15 SW_and_D, SW16 SW_and_D, SW17 SW_and_D, SW18 SW_and_D, SW19 SW_and_D, SW2 SW_and_D, SW20 SW_and_D, SW21 SW_and_D, SW22 SW_and_D, SW23 SW_and_D, SW24 SW_and_D, SW3 SW_and_D, SW4 SW_and_D, SW5 SW_and_D, SW6 SW_and_D, SW7 SW_and_D, SW8 SW_and_D, SW9 SW_and_D, U1 ProMicro/BLEMicroPro, U2 ProMicro/BLEMicroPro

Commit message: Replaced with stable version
Parts:
- SW1, SW10, SW11, SW12, SW13, SW14, SW15, SW16, SW17, SW18, SW19, SW2, SW20, SW21, SW22, SW23, SW24, SW3, SW4, SW5, SW6, SW7, SW8, SW9: footprint #footprint:CherryMX_MidHeight_Choc_16mm_rev8 -> #footprint:CherryMX_MidHeight_Choc_16mm_rev7
Routing:
- net Y2: track 330.6 -> 333.2 mm
- net Y6: track 403.4 -> 402.6 mm
- net Y5: track 277.5 -> 276.8 mm
- net Y3: track 278.8 -> 278.2 mm
- net Y4: track 271.9 -> 271.3 mm
Other:
- board text added: "stagger"
- board text added: "te96 Rev.2 by @e3w2q"
- board text removed: "0.2"
- board text removed: "0.25"
- board text removed: "0.3"
- board text removed: "0.35"
- board text removed: "0.4"
- board text removed: "0.45"
- board text removed: "4.8"
- board text removed: "4.9"
- board text removed: "5"
- board text removed: "5.1"
- board text removed: "A1"
- board text removed: "A2"
- board text removed: "A3"
- board text removed: "A4"
- board text removed: "A5"
- board text removed: "A6"
- board text removed: "B1"
- board text removed: "C1"
- board text removed: "D1"
- board text removed: "te96 Rev.3 by @e3w2q"

Commit message: Rev.3
Parts:
- SW1, SW10, SW11, SW12, SW13, SW14, SW15, SW16, SW17, SW18, SW19, SW2, SW20, SW21, SW22, SW23, SW24, SW3, SW4, SW5, SW6, SW7, SW8, SW9: footprint #footprint:CherryMX_MidHeight_Choc_16mm_rev7 -> #footprint:CherryMX_MidHeight_Choc_16mm_rev8
Routing:
- net Y2: track 333.2 -> 330.6 mm
- net Y6: track 402.6 -> 403.4 mm
- net Y5: track 276.8 -> 277.5 mm
- net Y3: track 278.2 -> 278.8 mm
- net Y4: track 271.3 -> 271.9 mm
Other:
- board text added: "A1"
- board text added: "A2"
- board text added: "A3"
- board text added: "A4"
- board text added: "A5"
- board text added: "A6"
- board text added: "B1"
- board text added: "C1"
- board text added: "D1"
- board text added: "te96 Rev.3 by @e3w2q"
- board text removed: "stagger"
- board text removed: "te96 Rev.2 by @e3w2q"

Commit message: Rev.4
Other:
- board text added: "te96 Rev.4 by @e3w2q"
- board text removed: "te96 Rev.3 by @e3w2q"

Commit message: Rev.5
Other:
- board text added: "te96 Rev.5 by @e3w2q"
- board text removed: "te96 Rev.4 by @e3w2q"
