File: pcb/te96.sch (KiCad schematic (older format))
At the start: 34 parts, among them J1 Conn_02x08_Top_Bottom, J10 Conn_01x04, J2 Conn_02x08_Top_Bottom, J3 MJ-4PP-9, J4 MJ-4PP-9, J7 Conn_01x03, J8 Conn_01x03, J9 Conn_01x04, SW1 SW_and_D, SW10 SW_and_D, SW11 SW_and_D, SW12 SW_and_D, SW13 SW_and_D, SW14 SW_and_D, SW15 SW_and_D, SW16 SW_and_D, SW17 SW_and_D, SW18 SW_and_D, SW19 SW_and_D, SW2 SW_and_D, SW20 SW_and_D, SW21 SW_and_D, SW22 SW_and_D, SW23 SW_and_D, SW24 SW_and_D, SW3 SW_and_D, SW4 SW_and_D, SW5 SW_and_D, SW6 SW_and_D, SW7 SW_and_D, SW8 SW_and_D, SW9 SW_and_D, U1 ProMicro/BLEMicroPro, U2 ProMicro/BLEMicroPro

Commit message: Replaced with stable version
Parts:
- SW1, SW10, SW11, SW12, SW13, SW14, SW15, SW16, SW17, SW18, SW19, SW2, SW20, SW21, SW22, SW23, SW24, SW3, SW4, SW5, SW6, SW7, SW8, SW9: footprint #footprint:CherryMX_MidHeight_Choc_16mm_rev8 -> #footprint:CherryMX_MidHeight_Choc_16mm_rev5
Changed lines of the file:
@@
 Title "te96 Sukeroku Keyboard"
 Date ""
-Rev "3"
+Rev "2"
 Comp "@e3w2q"
 Comment1 ""
@@
 F 0 "SW1" H 10828 1700 50  0000 L CNN
 F 1 "SW_and_D" H 10828 1609 50  0000 L CNN
-F 2 "#footprint:CherryMX_MidHeight_Choc_16mm_rev8" H 10550 1950 50  0001 C CNN
+F 2 "#footprint:CherryMX_MidHeight_Choc_16mm_rev5" H 10550 1950 50  0001 C CNN
 F 3 "" H 10550 1950 50  0001 C CNN
 	1    10550 1750
@@
 F 0 "SW7" H 9778 1700 50  0000 L CNN
 F 1 "SW_and_D" H 9778 1609 50  0000 L CNN
-F 2 "#footprint:CherryMX_MidHeight_Choc_16mm_rev8" H 9500 1950 50  0001 C CNN
+F 2 "#footprint:CherryMX_MidHeight_Choc_16mm_rev5" H 9500 1950 50  0001 C CNN
 F 3 "" H 9500 1950 50  0001 C CNN
 	1    9500 1750
@@
 F 0 "SW13" H 8678 1700 50  0000 L CNN
 F 1 "SW_and_D" H 8678 1609 50  0000 L CNN
-F 2 "#footprint:CherryMX_MidHeight_Choc_16mm_rev8" H 8400 1950 50  0001 C CNN
+F 2 "#footprint:CherryMX_MidHeight_Choc_16mm_rev5" H 8400 1950 50  0001 C CNN
 F 3 "" H 8400 1950 50  0001 C CNN
 	1    8400 1750
@@
 F 0 "SW19" H 7628 1700 50  0000 L CNN
 F 1 "SW_and_D" H 7628 1609 50  0000 L CNN
-F 2 "#footprint:CherryMX_MidHeight_Choc_16mm_rev8" H 7350 1950 50  0001 C CNN
+F 2 "#footprint:CherryMX_MidHeight_Choc_16mm_rev5" H 7350 1950 50  0001 C CNN
 F 3 "" H 7350 1950 50  0001 C CNN
 	1    7350 1750
@@
 F 0 "SW2" H 10828 2300 50  0000 L CNN
 F 1 "SW_and_D" H 10828 2209 50  0000 L CNN
-F 2 "#footprint:CherryMX_MidHeight_Choc_16mm_rev8" H 10550 2550 50  0001 C CNN
+F 2 "#footprint:CherryMX_MidHeight_Choc_16mm_rev5" H 10550 2550 50  0001 C CNN
 F 3 "" H 10550 2550 50  0001 C CNN
 	1    10550 2350
@@
 F 0 "SW8" H 9778 2300 50  0000 L CNN
 F 1 "SW_and_D" H 9778 2209 50  0000 L CNN
-F 2 "#footprint:CherryMX_MidHeight_Choc_16mm_rev8" H 9500 2550 50  0001 C CNN
+F 2 "#footprint:CherryMX_MidHeight_Choc_16mm_rev5" H 9500 2550 50  0001 C CNN
 F 3 "" H 9500 2550 50  0001 C CNN
 	1    9500 2350
@@
 F 0 "SW20" H 7628 2300 50  0000 L CNN
 F 1 "SW_and_D" H 7628 2209 50  0000 L CNN
-F 2 "#footprint:CherryMX_MidHeight_Choc_16mm_rev8" H 7350 2550 50  0001 C CNN
+F 2 "#footprint:CherryMX_MidHeight_Choc_16mm_rev5" H 7350 2550 50  0001 C CNN
 F 3 "" H 7350 2550 50  0001 C CNN
 	1    7350 2350
@@
 F 0 "SW3" H 10828 2900 50  0000 L CNN
 F 1 "SW_and_D" H 10828 2809 50  0000 L CNN
-F 2 "#footprint:CherryMX_MidHeight_Choc_16mm_rev8" H 10550 3150 50  0001 C CNN
+F 2 "#footprint:CherryMX_MidHeight_Choc_16mm_rev5" H 10550 3150 50  0001 C CNN
 F 3 "" H 10550 3150 50  0001 C CNN
 	1    10550 2950
@@
 F 0 "SW9" H 9778 2900 50  0000 L CNN
 F 1 "SW_and_D" H 9778 2809 50  0000 L CNN
-F 2 "#footprint:CherryMX_MidHeight_Choc_16mm_rev8" H 9500 3150 50  0001 C CNN
+F 2 "#footprint:CherryMX_MidHeight_Choc_16mm_rev5" H 9500 3150 50  0001 C CNN
 F 3 "" H 9500 3150 50  0001 C CNN
 	1    9500 2950
@@
 F 0 "SW15" H 8678 2900 50  0000 L CNN
 F 1 "SW_and_D" H 8678 2809 50  0000 L CNN
-F 2 "#footprint:CherryMX_MidHeight_Choc_16mm_rev8" H 8400 3150 50  0001 C CNN
+F 2 "#footprint:CherryMX_MidHeight_Choc_16mm_rev5" H 8400 3150 50  0001 C CNN
 F 3 "" H 8400 3150 50  0001 C CNN
 	1    8400 2950
@@
 F 0 "SW21" H 7628 2900 50  0000 L CNN
 F 1 "SW_and_D" H 7628 2809 50  0000 L CNN
-F 2 "#footprint:CherryMX_MidHeight_Choc_16mm_rev8" H 7350 3150 50  0001 C CNN
+F 2 "#footprint:CherryMX_MidHeight_Choc_16mm_rev5" H 7350 3150 50  0001 C CNN
 F 3 "" H 7350 3150 50  0001 C CNN
 	1    7350 2950
@@
 F 0 "SW4" H 10828 3500 50  0000 L CNN
 F 1 "SW_and_D" H 10828 3409 50  0000 L CNN
-F 2 "#footprint:CherryMX_MidHeight_Choc_16mm_rev8" H 10550 3750 50  0001 C CNN
+F 2 "#footprint:CherryMX_MidHeight_Choc_16mm_rev5" H 10550 3750 50  0001 C CNN
 F 3 "" H 10550 3750 50  0001 C CNN
 	1    10550 3550
@@
 F 0 "SW10" H 9778 3500 50  0000 L CNN
 F 1 "SW_and_D" H 9778 3409 50  0000 L CNN
-F 2 "#footprint:CherryMX_MidHeight_Choc_16mm_rev8" H 9500 3750 50  0001 C CNN
+F 2 "#footprint:CherryMX_MidHeight_Choc_16mm_rev5" H 9500 3750 50  0001 C CNN
 F 3 "" H 9500 3750 50  0001 C CNN
 	1    9500 3550
@@
 F 0 "SW16" H 8678 3500 50  0000 L CNN
 F 1 "SW_and_D" H 8678 3409 50  0000 L CNN
-F 2 "#footprint:CherryMX_MidHeight_Choc_16mm_rev8" H 8400 3750 50  0001 C CNN
+F 2 "#footprint:CherryMX_MidHeight_Choc_16mm_rev5" H 8400 3750 50  0001 C CNN
 F 3 "" H 8400 3750 50  0001 C CNN
 	1    8400 3550
@@
 F 0 "SW22" H 7628 3500 50  0000 L CNN
 F 1 "SW_and_D" H 7628 3409 50  0000 L CNN
-F 2 "#footprint:CherryMX_MidHeight_Choc_16mm_rev8" H 7350 3750 50  0001 C CNN
+F 2 "#footprint:CherryMX_MidHeight_Choc_16mm_rev5" H 7350 3750 50  0001 C CNN
 F 3 "" H 7350 3750 50  0001 C CNN
 	1    7350 3550
@@
 F 0 "SW5" H 10828 4100 50  0000 L CNN
 F 1 "SW_and_D" H 10828 4009 50  0000 L CNN
-F 2 "#footprint:CherryMX_MidHeight_Choc_16mm_rev8" H 10550 4350 50  0001 C CNN
+F 2 "#footprint:CherryMX_MidHeight_Choc_16mm_rev5" H 10550 4350 50  0001 C CNN
 F 3 "" H 10550 4350 50  0001 C CNN
 	1    10550 4150
@@
 F 0 "SW11" H 9778 4100 50  0000 L CNN
 F 1 "SW_and_D" H 9778 4009 50  0000 L CNN
-F 2 "#footprint:CherryMX_MidHeight_Choc_16mm_rev8" H 9500 4350 50  0001 C CNN
+F 2 "#footprint:CherryMX_MidHeight_Choc_16mm_rev5" H 9500 4350 50  0001 C CNN
 F 3 "" H 9500 4350 50  0001 C CNN
 	1    9500 4150
@@
 F 0 "SW17" H 8678 4100 50  0000 L CNN
 F 1 "SW_and_D" H 8678 4009 50  0000 L CNN
-F 2 "#footprint:CherryMX_MidHeight_Choc_16mm_rev8" H 8400 4350 50  0001 C CNN
+F 2 "#footprint:CherryMX_MidHeight_Choc_16mm_rev5" H 8400 4350 50  0001 C CNN
 F 3 "" H 8400 4350 50  0001 C CNN
 	1    8400 4150
@@
 F 0 "SW23" H 7628 4100 50  0000 L CNN
 F 1 "SW_and_D" H 7628 4009 50  0000 L CNN
-F 2 "#footprint:CherryMX_MidHeight_Choc_16mm_rev8" H 7350 4350 50  0001 C CNN
+F 2 "#footprint:CherryMX_MidHeight_Choc_16mm_rev5" H 7350 4350 50  0001 C CNN
 F 3 "" H 7350 4350 50  0001 C CNN
 	1    7350 4150
@@
 F 0 "SW6" H 10828 4700 50  0000 L CNN
 F 1 "SW_and_D" H 10828 4609 50  0000 L CNN
-F 2 "#footprint:CherryMX_MidHeight_Choc_16mm_rev8" H 10550 4950 50  0001 C CNN
+F 2 "#footprint:CherryMX_MidHeight_Choc_16mm_rev5" H 10550 4950 50  0001 C CNN
 F 3 "" H 10550 4950 50  0001 C CNN
 	1    10550 4750
@@
 F 0 "SW12" H 9778 4700 50  0000 L CNN
 F 1 "SW_and_D" H 9778 4609 50  0000 L CNN
-F 2 "#footprint:CherryMX_MidHeight_Choc_16mm_rev8" H 9500 4950 50  0001 C CNN
+F 2 "#footprint:CherryMX_MidHeight_Choc_16mm_rev5" H 9500 4950 50  0001 C CNN
 F 3 "" H 9500 4950 50  0001 C CNN
 	1    9500 4750
@@
 F 0 "SW18" H 8678 4700 50  0000 L CNN
 F 1 "SW_and_D" H 8678 4609 50  0000 L CNN
-F 2 "#footprint:CherryMX_MidHeight_Choc_16mm_rev8" H 8400 4950 50  0001 C CNN
+F 2 "#footprint:CherryMX_MidHeight_Choc_16mm_rev5" H 8400 4950 50  0001 C CNN
 F 3 "" H 8400 4950 50  0001 C CNN
 	1    8400 4750
@@
 F 0 "SW24" H 7628 4700 50  0000 L CNN
 F 1 "SW_and_D" H 7628 4609 50  0000 L CNN
-F 2 "#footprint:CherryMX_MidHeight_Choc_16mm_rev8" H 7350 4950 50  0001 C CNN
+F 2 "#footprint:CherryMX_MidHeight_Choc_16mm_rev5" H 7350 4950 50  0001 C CNN
 F 3 "" H 7350 4950 50  0001 C CNN
 	1    7350 4750
@@
 F 0 "SW14" H 8678 2300 50  0000 L CNN
 F 1 "SW_and_D" H 8678 2209 50  0000 L CNN
-F 2 "#footprint:CherryMX_MidHeight_Choc_16mm_rev8" H 8400 2550 50  0001 C CNN
+F 2 "#footprint:CherryMX_MidHeight_Choc_16mm_rev5" H 8400 2550 50  0001 C CNN
 F 3 "" H 8400 2550 50  0001 C CNN
 	1    8400 2350

Commit message: Rev.3
Parts:
- SW1, SW10, SW11, SW12, SW13, SW14, SW15, SW16, SW17, SW18, SW19, SW2, SW20, SW21, SW22, SW23, SW24, SW3, SW4, SW5, SW6, SW7, SW8, SW9: footprint #footprint:CherryMX_MidHeight_Choc_16mm_rev5 -> #footprint:CherryMX_MidHeight_Choc_16mm_rev8
Other:
- moved on the sheet: J1, J10, J2, J3, J4, J7, J8, J9, SW1, SW10, SW11, SW12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
